Commit message: Modifying static tranform for 2D lidar

File: urdf/accessories/sick_lms1xx.urdf.xacro (robot description, xacro)
@@ -27,6 +27,6 @@
 <!-- Modified LiDAR parameters to match RPLiDAR A3 which is the one used by the physical robot -->
 <!-- Previous -->
-<xacro:macro name="sick_lms1xx" params="frame:=laser topic:=scan sample_size:=720 update_rate:=50
-               min_angle:=-2.35619 max_angle:=2.35619 min_range:=0.1 max_range:=30.0 robot_namespace:=/" >
+<!--<xacro:macro name="sick_lms1xx" params="frame:=laser topic:=scan sample_size:=720 update_rate:=50
+               min_angle:=-2.35619 max_angle:=2.35619 min_range:=0.1 max_range:=30.0 robot_namespace:=/" >-->
 <robot xmlns:xacro="http://www.ros.org/wiki/xacro">
   <!-- New RPLiDR A3 obtained from: https://github.com/husarion/rosbot_description/blob/master/src/rosbot_description/urdf/rosbot.gazebo -->
